Commit message: created rough urdf of test bot with lms111 mesh

File: urdf/test_bot.urdf (robot description, URDF)
Before this commit: robot sam_bot, 0 links, 0 joints
Links:
- added link base_laser; visual mesh filename=package://officebot_description/meshes/LMS111.stl
- added link base_link
- added link bot_base; visual box size=${base_length} ${base_width} ${base_height}
Joints:
- added joint base_height: type fixed, parent base_link, child bot_base, origin xyz=0 0 0.05 rpy=0 0 0
- added joint laser_link: type fixed, parent bot_base, child base_laser, origin xyz=0 0 0.19 rpy=0 0 0

Commit message: added in wheels for the test bot

File: urdf/test_bot.urdf (robot description, URDF)
Before this commit: robot test_bot, 3 links, 2 joints
Links:
- added link left_wheel_link; visual cylinder length=0.05 radius=${wheel_diameter/2}
- added link right_wheel_link; visual cylinder length=0.05 radius=${wheel_diameter/2}
Joints:
- added joint left_wheel_joint: type fixed, parent bot_base, child left_wheel_link, origin xyz=0 ${wheel_y_offset} -${wheel_diameter/2} rpy=0 0 0
- added joint right_wheel_joint: type fixed, parent bot_base, child right_wheel_link, origin xyz=0 -${wheel_y_offset} -${wheel_diameter/2} rpy=0 0 0
- joint base_height: origin xyz=0 0 0.05 rpy=0 0 0 -> xyz=0 0 0.0624 rpy=0 0 0
