Commit message: Added in base_laser frame and top sensor link frame.

File: urdf/ot_bot.urdf (robot description, URDF)
Before this commit: robot office_bot, 2 links, 1 joints
Links:
- added link base_laser; visual mesh filename=package://officebot_description/meshes/sick_tim_571.stl
- added link sensor_plate_link
Joints:
- added joint botbottom_to_topsensorplate: type fixed, parent bot_base, child sensor_plate_link, origin xyz=0 0 0.476 rpy=0 0 0
- added joint topsensorplate_to_base_laser: type fixed, parent sensor_plate_link, child base_laser, origin xyz=0 0 0.07246 rpy=0 0 0
- joint base_height: origin xyz=0 0 0.0624 rpy=0 0 0 -> xyz=0 0 0.0645 rpy=0 0 0
